Commit message: update grasping params

File: data_urdf/object/contactdb/sphere_tennis/coacd_decomposed_object_one_link.urdf (robot description, URDF)
Before this commit: robot sphere_tennis, 1 links, 0 joints
Links:
- link object: geometry collision mesh filename=coacd_allinone.obj scale=1.0000E+00 1.0000E+00 1.0000E+00; visual mesh filename=sphere_tennis.stl scale=1.0000E+00 1.0000E+00 1.0000E+00
